File: breakout-tt08-cob.kicad_pcb (KiCad board)
At the start: 2 copper layers, 50 x 52 mm, 157 parts, among them CON1 NPTC202KFMS-RC, CON2 NPTC202KFMS-RC, J1 Conn_01x04, J2 Conn_02x06_Odd_Even, J3 Conn_02x06_Odd_Even, U1 Openframe_QFN_TT06_REV2, U2 24LC02

Commit message: update metadata and production export settings
Parts:
- U1: value Openframe_QFN_TT06_REV2 -> Openframe_COB_TT08
Changed lines of the file:
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@@
 	(paper "User" 140.005 119.99)
 	(title_block
-		(title "Tiny Tapeout 06+ Breakout QFN")
-		(date "2025-02-24")
-		(rev "2.0")
-		(company "Psychogenic Technologies")
-		(comment 1 "(C) 2025 Pat Deegan")
+		(title "Tiny Tapeout 8 COB breakout")
+		(date "2025-10-28")
+		(rev "1.0")
+		(comment 1 "Based on psychogenic's QFN breakout")
 	)
 	(layers
@@
 			)
 		)
-		(property "Value" "Openframe_QFN_TT06_REV2"
+		(property "Value" "Openframe_COB_TT08"
 			(at 0 6.5 180)
 			(unlocked yes)
@@
 			)
 		)
-		(property "Datasheet" "https://github.com/TinyTapeout/tt-multiplexer/blob/tt06-staging/docs/INFO.md#pinout"
+		(property "Datasheet" "https://github.com/TinyTapeout/tt-multiplexer/blob/tt08-release/docs/INFO.md#pinout"
 			(at 0 0 180)
 			(unlocked yes)
@@
 			)
 		)
-		(property "Description" "Openframe QFN packaging, with TinyTapeout 6+ pin mapping"
+		(property "Description" ""
 			(at 0 0 180)
 			(unlocked yes)
@@
 		)
 		(group ""
-			(members "1c26c2e7-0a4b-4265-b1ed-631bb8872b56" "b63cd45f-28d8-433a-8ba1-6931475cffde")
+			(members "80284a78-fd9b-4b13-8fce-5242b75c16ae" "8380e97b-c5a9-4698-b6d6-fa2b72237934")
 		)
 		(group ""
-			(members "9d63aea4-6e8d-431b-9c32-c2a31dcd1e78")
+			(members "403384ce-c7d4-4fec-8ffc-ff4b56653a0f")
 		)
 		(group ""
-			(members "029918d2-f316-4acd-8d2d-411a2ab378c3" "2af85737-aa4c-4f7b-b414-3d5ef1c77807"
-				"3fa73dda-ae4e-43f7-a736-9f351c3c6174" "5a5c1003-e564-4a40-a831-9f8316588b42"
-				"8ffb9985-e269-49b5-84c6-bcf47e08201c" "da51e61f-b064-4549-a0db-7f5659f56452"
-				"dc524304-82f4-4f30-8ddd-007623882a45" "ecd7b6ef-1e98-45d6-8fbb-5206591fe1a5"
+			(members "0a858087-04d6-4d87-a896-c1c62366076b" "372ec213-bd3d-42ff-ab7b-cde2728bab74"
+				"56aa6ae0-89ea-499b-bf85-8381652556ed" "6743290b-8aa2-494e-9b84-1e0ed1221c81"
+				"7ac34704-0dd1-4618-a214-f220d4660e72" "9bb166a2-1a38-4702-938e-6c47a43885ce"
+				"9e42c8cd-e3af-463e-b1de-c47e0baf1de5" "ed0702d0-77b6-4c45-be58-22100d45e56b"
 			)
 		)
 		(group ""
-			(members "0030e167-b449-444f-b814-764f14d00e63" "0381ac5f-a1dc-49fa-9ac4-e4dacf3939db"
-				"08b194c1-c6a7-43f9-a77b-f9401238b3c9" "0b3c5121-f950-41b0-882f-b62b138bc938"
-				"0e9212e6-2ebe-49c6-844b-a5d55ef675c9" "11e74bed-92e4-4437-aa7f-d648175fd104"
-				"1400cdd2-f90c-471f-b2cd-d0b0a7487559" "1427e161-df22-4c99-845b-0e02f163735f"
-				"18c3c4fe-a40b-4f21-9d6f-91f7ef0afbbb" "1957e574-ee33-4796-86ca-04a854a93419"
-				"1ab616c3-7a07-4164-a47f-30c9cd8ceb27" "1db86d7f-4404-40c5-9e6e-41d2a79d93ed"
-				"1df611e6-d27d-4e34-9ec8-32f172f84df9" "204ec7ad-96e2-4a9b-8c8e-3c61a3acc579"
-				"26aceb9d-4759-452a-b68a-8d3e3f289b16" "27373bca-876c-4c99-82f4-bf20e1754807"
-				"2f7362e3-e9ee-4336-8417-80d689d1d96d" "3258541e-33a0-419c-84da-358e9c5da68e"
-				"32c83cbb-a2dd-4593-8838-df04757b0e2c" "369f837a-ef57-4e22-bfe5-036bea5c125e"
-				"372c444f-15f4-4f08-b658-da602d75f287" "39f4e778-c4a4-4edd-a32f-964e7724cd05"
-				"45a4858e-cc32-410f-9025-607843477844" "4a6aeff2-bda3-4390-8c91-3940a9e037bc"
-				"54325f0f-f020-4732-8149-47dadf76d706" "5ba7c66e-3e36-4027-83e1-5af90b5a9482"
-				"691eb7b9-ecae-442c-931d-d513577e8ffa" "756493fe-6ce1-4ace-829f-c71eb4a99d14"
-				"7590265a-d097-448a-881c-4fd1eb25b7ee" "7e430358-19e6-4400-94e7-cb4f1b8c629d"
-				"8055a53a-efb3-4245-af0c-1bebb8232f31" "80b248c0-f4af-4162-9d98-35394817960c"
-				"82870faf-4076-4d78-abee-df4132029dd4" "8ad3808d-b670-4761-9b50-f345b1f6d95c"
-				"908e62e9-86c5-4788-9e9b-4410c8d86d6f" "909dea03-07a7-436a-9e21-104fddd04ae3"
-				"9e3bbad5-e248-41dd-9356-a4fb3fca0966" "9e5f579a-7c22-4491-8954-f54966530d41"
-				"a2a71326-1b20-4bd3-b6d3-e2d26d21cd2a" "a5fcd344-08ba-4260-851d-517fe0aeadba"
-				"a60fcf02-c786-4c00-a822-67f155964019" "a8b04412-ba4f-4e26-b8fd-5618990785e2"
-				"ac686e24-733c-4fde-8a01-b55b5eb6eff8" "adeff426-03c4-49f8-87b9-5349a7d6b357"
-				"b3c6e829-a132-4fbd-a623-ef68c42c0a23" "b692775a-fac3-410c-bfec-5f702a668585"
-				"bd6f850c-c51f-4cfc-ad69-cde25707d3ab" "c03e8987-dbb9-4cf6-afc4-6e3cca54ac8a"
-				"c13e8e8d-444e-41ad-a659-276738de82e6" "c3c96bec-c500-4074-9d8e-9078452ff8d2"
-				"ca644787-6a05-4b31-afae-e19853d55165" "cbafbb4c-dac7-4864-adce-08fe3faeac58"
-				"cca59039-7f2c-4bb7-a122-c83bc172fd8b" "d30cf442-cb91-4e0f-a341-7699bdaf17d5"
-				"d82fb585-fe44-49ba-84fc-381bf79a94c6" "da0c3afa-e2c1-457f-8411-2f6ca7be9ec8"
-				"dc61831d-401d-4bb2-925a-dc8bc0d6c919" "e6b844a6-8b8d-41e8-9d18-47643f99901d"
-				"e9377930-0d8b-4a52-989d-6ba59306710a" "ee624758-22be-46eb-a1aa-f8538e1d298c"
-				"f2c51d36-e942-416a-b812-c20d96fb24a7" "f308e411-96d5-4b01-93f8-7b08e1046f40"
-				"f958dab9-2bbf-436e-b7bb-7721b28ab6b3" "fdab15ac-2f76-4462-9883-7a978c73226e"
+			(members "065c9922-08e1-4ac6-86f5-55c0a56e1999" "083da663-2107-400c-abb5-586575c315b3"
+				"0fccfb32-ea3b-4213-852c-d803415cbf19" "11b9ceaa-517c-4b9e-8fe7-6305b46ebc49"
+				"1b9ed62b-25d3-4cb3-b694-b7037b9ae8b3" "20eb3482-5dd0-410c-b5a2-add49800d01d"
+				"290c00d9-4297-428a-92d6-9b502115dba9" "29a756c2-301d-42e0-992e-c9f83d4a3162"
+				"2fba32da-0f1c-4244-8879-7dc61a60ea1a" "31c2f6d1-5ce2-48e3-aafe-4e297edb9e3b"
+				"373dc8e3-d573-4416-b6a5-03e6c35b3f9b" "3d931745-d612-4ae0-90aa-98ca32926ea8"
+				"3eab3e8c-dcb5-42cf-bc34-ccef6e57edae" "40cce340-6803-4e54-bc19-9097ba23fadf"
+				"46d3c936-77f0-4d3e-a8db-cc535d4ca310" "49d474f5-818f-466f-8f95-e6dbcae27f95"
+				"4e8fe841-b23c-45d5-8008-74f8217dc082" "53b27c8e-6d6d-4fee-b645-6f8dafc797cc"
+				"547ddaa8-6465-4e84-bc3d-83f1ba593572" "5745651d-e8aa-4b16-b3c5-7e4104fc2391"
+				"57e885fe-21aa-4b22-86a6-0909ecbaf466" "59227de5-95bd-4009-915a-769f0a05ad14"
+				"5c01aa1d-ca1f-430f-a93d-58f2462e2025" "5ee0b5de-8acf-44f5-acf9-35967b43d1d1"
+				"6244dcba-a06b-40b5-8960-eb2bc7d28771" "6a81074a-45dd-492b-abd7-49ffbd7abb98"
+				"6c1d0627-821d-47a3-81e6-5d3a4ee8b540" "6d4ad1d4-ef70-4f73-9cf2-5edf94a8f06f"
+				"6ddaead0-0b82-4e31-b2a9-a07c1c94c7f6" "6f56738d-c7ea-4c74-8b6f-f60a43cafe78"
+				"6fe7ccd3-4dec-415a-b5cc-1af477029522" "7cfd7a50-196b-42e8-a976-2f784b954198"
+				"81829161-f254-4d93-b1eb-cc07303eb23f" "8a299338-332e-4faa-a92f-e520193b2efc"
+				"8d26ee52-d298-4d83-8bf7-7260e1b320a0" "8dc9e608-1691-48ed-a31e-b403e8d2509d"
+				"90bdb5df-8c0b-4d1e-b4ba-7b104bc63c3c" "946944fe-9a69-4887-a431-dcf6ab835ae0"
+				"97c984ec-48ed-4af5-aa70-0d92dab08078" "9c2a1228-6aab-4937-9ba3-2146b8b5fe65"
+				"9c5fe137-dfcb-4fe1-818e-d53ed76eeca6" "a385e7c8-72f5-4b7f-bb39-49973a981418"
+				"a6e8bb1f-1c5a-455e-aa92-bf61a0698ee9" "acbaa95c-fd55-4b80-84dd-cf8a0bb68d6e"
+				"aea5004a-a4a0-4da8-84b0-b85594b8e414" "afabafe2-0a5c-45fa-9247-f8f270e8518d"
+				"b2a1ad74-d501-4bc9-90b2-81cea2c05234" "b9e36f34-e751-49a8-a092-733be6d9c216"
+				"ba62bee0-30bf-45be-9488-26b6cfa1d0b1" "bdfbaef4-fee9-4d11-aaae-73d00fceac0c"
+				"c24a4df7-2024-493c-9012-4a84747ccce2" "c66d44f8-41dc-4671-bdf3-15c7765566f3"
+				"c6d9eb23-bfa5-4cc1-a4b3-015fdb0da8e5" "ce4367bb-223b-4638-a41b-ea181a94e54e"
+				"d263a490-5984-413f-80d9-86ab8038f656" "d60d0ca4-085c-4c5a-9ef9-7d6af5961f3d"
+				"d7212a17-45c9-4e87-929d-397d05fe560b" "dcf9b668-0ee5-4bed-8246-f7f72fc9dcf1"
+				"e2fb9a23-5aaf-4c83-a3e8-6311f4d10c4e" "e9146811-e207-4e81-bae3-04186d600d7f"
+				"eadd0058-a2be-4841-9e97-86b27770a7e1" "f9339b1e-9704-478b-927c-2be0f5acb844"
+				"fb56752f-223b-411d-a120-225863897c05" "fe540985-197c-48e4-b81c-46757f27e611"
 			)
 		)
