File: breakout-tt08-cob.kicad_sch (KiCad schematic)
At the start: 58 parts, among them CON1 NPTC202KFMS-RC, CON2 NPTC202KFMS-RC, J1 Conn_01x04, J2 Conn_02x06_Odd_Even, J3 Conn_02x06_Odd_Even, U1 Openframe_QFN_TT06_REV2, U2 24LC02

Commit message: update metadata and production export settings
Parts:
- U1: value Openframe_QFN_TT06_REV2 -> Openframe_COB_TT08
Changed lines of the file:
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@@
 			)
 		)
-		(property "Value" "Openframe_QFN_TT06_REV2"
+		(property "Value" "Openframe_COB_TT08"
 			(at 117.856 123.19 90)
 			(effects
@@
 			)
 		)
-		(property "Datasheet" "https://github.com/TinyTapeout/tt-multiplexer/blob/tt06-staging/docs/INFO.md#pinout"
+		(property "Datasheet" "https://github.com/TinyTapeout/tt-multiplexer/blob/tt08-release/docs/INFO.md#pinout"
 			(at 142.24 92.71 0)
 			(effects
@@
 			)
 		)
-		(property "Description" "Openframe QFN packaging, with TinyTapeout 6+ pin mapping"
+		(property "Description" ""
 			(at 91.44 95.25 0)
 			(effects
